File: schematics/bracelet/Bracelet.sch (EAGLE design)
At the start: 14 parts

Commit message: finished layout, accel pullups need to be conf'ed to internal.
Parts:
- removed R4, R5: 1k, rcl:R-EU_R0805
Connections:
- removed net VDDIO: R4.2, R5.1
- net CAP01: now also U$1.P15_A1_CS4; no longer U$1.P23_A9_CS2
- net CAP03: now also U$1.P16_A2_SCL
- net CAP05: now also U$1.P17_A3_SDA; no longer U$1.P22_A8_CS3
- net CAP06: no longer U$1.P15_A1_CS4
- net CAP07: now also U$1.P23_A9_CS2; no longer U$1.P17_A3_SDA
- net CAP08: now also U$1.P22_A8_CS3; no longer U$1.P16_A2_SCL
- net SCL: no longer R4.1
- net SDA: no longer R5.2
Changed lines of the file:
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@@
 <part name="GND9" library="supply1" deviceset="GND" device=""/>
 <part name="GND10" library="supply1" deviceset="GND" device=""/>
-<part name="R4" library="rcl" deviceset="R-EU_" device="R0805" value="1k"/>
-<part name="R5" library="rcl" deviceset="R-EU_" device="R0805" value="1k"/>
 <part name="C1" library="rcl" deviceset="C-EU" device="C0805" value="1uF"/>
 <part name="C2" library="rcl" deviceset="C-EU" device="C0805" value="0.1uF"/>
@@
 <part name="C4" library="rcl" deviceset="C-EU" device="C0805" value="0.1uF"/>
 <part name="+3V4" library="supply1" deviceset="+3V3" device=""/>
-<part name="+3V5" library="supply1" deviceset="+3V3" device=""/>
-<part name="+3V6" library="supply1" deviceset="+3V3" device=""/>
 </parts>
 <sheets>
@@
 <instance part="GND9" gate="1" x="-63.5" y="-2.54"/>
 <instance part="GND10" gate="1" x="-20.32" y="2.54"/>
-<instance part="R4" gate="G$1" x="-81.28" y="35.56" rot="R180"/>
-<instance part="R5" gate="G$1" x="-20.32" y="33.02" rot="R270"/>
 <instance part="C1" gate="G$1" x="-86.36" y="20.32"/>
 <instance part="C2" gate="G$1" x="-76.2" y="20.32"/>
@@
 <instance part="C4" gate="G$1" x="-20.32" y="15.24"/>
 <instance part="+3V4" gate="G$1" x="-10.16" y="20.32" rot="R270"/>
-<instance part="+3V5" gate="G$1" x="-101.6" y="35.56" rot="R90"/>
-<instance part="+3V6" gate="G$1" x="-5.08" y="40.64" rot="R270"/>
 </instances>
 <busses>
@@
 </segment>
 <segment>
+<pinref part="U$1" gate="G$1" pin="P15_A1_CS4"/>
+<wire x1="86.36" y1="71.12" x2="101.6" y2="71.12" width="0.1524" layer="91"/>
+<label x="93.98" y="71.12" size="1.778" layer="95"/>
+</segment>
+</net>
+<net name="CAP02" class="0">
+<segment>
+<pinref part="TOUCHSLIDER_CONNECTOR" gate="-2" pin="S"/>
+<wire x1="-66.04" y1="149.86" x2="-35.56" y2="149.86" width="0.1524" layer="91"/>
+<label x="-43.18" y="149.86" size="1.778" layer="95"/>
+</segment>
+<segment>
+<pinref part="U$1" gate="G$1" pin="P0_RX1"/>
+<wire x1="20.32" y1="121.92" x2="7.62" y2="121.92" width="0.1524" layer="91"/>
+<label x="7.62" y="121.92" size="1.778" layer="95"/>
+</segment>
+</net>
+<net name="CAP03" class="0">
+<segment>
+<pinref part="TOUCHSLIDER_CONNECTOR" gate="-3" pin="S"/>
+<wire x1="-66.04" y1="147.32" x2="-35.56" y2="147.32" width="0.1524" layer="91"/>
+<label x="-43.18" y="147.32" size="1.778" layer="95"/>
+</segment>
+<segment>
+<pinref part="U$1" gate="G$1" pin="P16_A2_SCL"/>
+<wire x1="86.36" y1="76.2" x2="101.6" y2="76.2" width="0.1524" layer="91"/>
+<label x="93.98" y="76.2" size="1.778" layer="95"/>
+</segment>
+</net>
+<net name="CAP04" class="0">
+<segment>
+<pinref part="TOUCHSLIDER_CONNECTOR" gate="-4" pin="S"/>
+<wire x1="-66.04" y1="144.78" x2="-35.56" y2="144.78" width="0.1524" layer="91"/>
+<label x="-43.18" y="144.78" size="1.778" layer="95"/>
+</segment>
+<segment>
+<pinref part="U$1" gate="G$1" pin="P1_TX1"/>
+<wire x1="20.32" y1="116.84" x2="7.62" y2="116.84" width="0.1524" layer="91"/>
+<label x="7.62" y="116.84" size="1.778" layer="95"/>
+</segment>
+</net>
+<net name="CAP05" class="0">
+<segment>
+<pinref part="TOUCHSLIDER_CONNECTOR" gate="-5" pin="S"/>
+<wire x1="-66.04" y1="142.24" x2="-35.56" y2="142.24" width="0.1524" layer="91"/>
+<label x="-43.18" y="142.24" size="1.778" layer="95"/>
+</segment>
+<segment>
+<pinref part="U$1" gate="G$1" pin="P17_A3_SDA"/>
+<wire x1="86.36" y1="81.28" x2="101.6" y2="81.28" width="0.1524" layer="91"/>
+<label x="93.98" y="81.28" size="1.778" layer="95"/>
+</segment>
+</net>
+<net name="CAP06" class="0">
+<segment>
+<pinref part="TOUCHSLIDER_CONNECTOR" gate="-6" pin="S"/>
+<wire x1="-66.04" y1="139.7" x2="-35.56" y2="139.7" width="0.1524" layer="91"/>
+<label x="-43.18" y="139.7" size="1.778" layer="95"/>
+</segment>
+</net>
+<net name="CAP07" class="0">
+<segment>
+<pinref part="TOUCHSLIDER_CONNECTOR" gate="-7" pin="S"/>
+<wire x1="-66.04" y1="137.16" x2="-35.56" y2="137.16" width="0.1524" layer="91"/>
+<label x="-43.18" y="137.16" size="1.778" layer="95"/>
+</segment>
+<segment>
 <pinref part="U$1" gate="G$1" pin="P23_A9_CS2"/>
 <wire x1="86.36" y1="111.76" x2="101.6" y2="111.76" width="0.1524" layer="91"/>
@@
 </segment>
 </net>
-<net name="CAP02" class="0">
-<segment>
-<pinref part="TOUCHSLIDER_CONNECTOR" gate="-2" pin="S"/>
-<wire x1="-66.04" y1="149.86" x2="-35.56" y2="149.86" width="0.1524" layer="91"/>
-<label x="-43.18" y="149.86" size="1.778" layer="95"/>
-</segment>
-<segment>
-<pinref part="U$1" gate="G$1" pin="P0_RX1"/>
-<wire x1="20.32" y1="121.92" x2="7.62" y2="121.92" width="0.1524" layer="91"/>
-<label x="7.62" y="121.92" size="1.778" layer="95"/>
-</segment>
-</net>
-<net name="CAP03" class="0">
-<segment>
-<pinref part="TOUCHSLIDER_CONNECTOR" gate="-3" pin="S"/>
-<wire x1="-66.04" y1="147.32" x2="-35.56" y2="147.32" width="0.1524" layer="91"/>
-<label x="-43.18" y="147.32" size="1.778" layer="95"/>
-</segment>
-</net>
-<net name="CAP04" class="0">
-<segment>
-<pinref part="TOUCHSLIDER_CONNECTOR" gate="-4" pin="S"/>
-<wire x1="-66.04" y1="144.78" x2="-35.56" y2="144.78" width="0.1524" layer="91"/>
-<label x="-43.18" y="144.78" size="1.778" layer="95"/>
-</segment>
-<segment>
-<pinref part="U$1" gate="G$1" pin="P1_TX1"/>
-<wire x1="20.32" y1="116.84" x2="7.62" y2="116.84" width="0.1524" layer="91"/>
-<label x="7.62" y="116.84" size="1.778" layer="95"/>
-</segment>
-</net>
-<net name="CAP05" class="0">
-<segment>
-<pinref part="TOUCHSLIDER_CONNECTOR" gate="-5" pin="S"/>
-<wire x1="-66.04" y1="142.24" x2="-35.56" y2="142.24" width="0.1524" layer="91"/>
-<label x="-43.18" y="142.24" size="1.778" layer="95"/>
+<net name="CAP08" class="0">
+<segment>
+<pinref part="TOUCHSLIDER_CONNECTOR" gate="-8" pin="S"/>
+<wire x1="-66.04" y1="134.62" x2="-35.56" y2="134.62" width="0.1524" layer="91"/>
+<label x="-43.18" y="134.62" size="1.778" layer="95"/>
 </segment>
 <segment>
@@
 <wire x1="86.36" y1="106.68" x2="101.6" y2="106.68" width="0.1524" layer="91"/>
 <label x="93.98" y="106.68" size="1.778" layer="95"/>
-</segment>
-</net>
-<net name="CAP06" class="0">
-<segment>
-<pinref part="TOUCHSLIDER_CONNECTOR" gate="-6" pin="S"/>
-<wire x1="-66.04" y1="139.7" x2="-35.56" y2="139.7" width="0.1524" layer="91"/>
-<label x="-43.18" y="139.7" size="1.778" layer="95"/>
-</segment>
-<segment>
-<pinref part="U$1" gate="G$1" pin="P15_A1_CS4"/>
-<wire x1="86.36" y1="71.12" x2="101.6" y2="71.12" width="0.1524" layer="91"/>
-<label x="93.98" y="71.12" size="1.778" layer="95"/>
-</segment>
-</net>
-<net name="CAP07" class="0">
-<segment>
-<pinref part="TOUCHSLIDER_CONNECTOR" gate="-7" pin="S"/>
-<wire x1="-66.04" y1="137.16" x2="-35.56" y2="137.16" width="0.1524" layer="91"/>
-<label x="-43.18" y="137.16" size="1.778" layer="95"/>
-</segment>
-<segment>
-<pinref part="U$1" gate="G$1" pin="P17_A3_SDA"/>
-<wire x1="86.36" y1="81.28" x2="101.6" y2="81.28" width="0.1524" layer="91"/>
-<label x="93.98" y="81.28" size="1.778" layer="95"/>
-</segment>
-</net>
-<net name="CAP08" class="0">
-<segment>
-<pinref part="TOUCHSLIDER_CONNECTOR" gate="-8" pin="S"/>
-<wire x1="-66.04" y1="134.62" x2="-35.56" y2="134.62" width="0.1524" layer="91"/>
-<label x="-43.18" y="134.62" size="1.778" layer="95"/>
-</segment>
-<segment>
-<pinref part="U$1" gate="G$1" pin="P16_A2_SCL"/>
-<wire x1="86.36" y1="76.2" x2="101.6" y2="76.2" width="0.1524" layer="91"/>
-<label x="93.98" y="76.2" size="1.778" layer="95"/>
 </segment>
 </net>
@@
 <segment>
 <pinref part="U$3" gate="G$1" pin="SDA"/>
-<pinref part="R5" gate="G$1" pin="2"/>
 <wire x1="-33.02" y1="25.4" x2="-20.32" y2="25.4" width="0.1524" layer="91"/>
 <wire x1="-20.32" y1="25.4" x2="-20.32" y2="27.94" width="0.1524" layer="91"/>
@@
 </segment>
 </net>
-<net name="VDDIO" class="0">
-<segment>
-<pinref part="R5" gate="G$1" pin="1"/>
-<wire x1="-20.32" y1="38.1" x2="-20.32" y2="40.64" width="0.1524" layer="91"/>
-<wire x1="-20.32" y1="40.64" x2="-7.62" y2="40.64" width="0.1524" layer="91"/>
-<label x="-15.24" y="40.64" size="1.778" layer="95"/>
-<pinref part="+3V6" gate="G$1" pin="+3V3"/>
-</segment>
-<segment>
-<pinref part="R4" gate="G$1" pin="2"/>
-<wire x1="-86.36" y1="35.56" x2="-99.06" y2="35.56" width="0.1524" layer="91"/>
-<label x="-99.06" y="35.56" size="1.778" layer="95"/>
-<pinref part="+3V5" gate="G$1" pin="+3V3"/>
-</segment>
-</net>
 <net name="SCL" class="0">
 <segment>
@@
 <wire x1="-68.58" y1="30.48" x2="-99.06" y2="30.48" width="0.1524" layer="91"/>
 <label x="-99.06" y="30.48" size="1.778" layer="95"/>
-<pinref part="R4" gate="G$1" pin="1"/>
-<wire x1="-76.2" y1="35.56" x2="-68.58" y2="35.56" width="0.1524" layer="91"/>
-<wire x1="-68.58" y1="35.56" x2="-68.58" y2="30.48" width="0.1524" layer="91"/>
-<junction x="-68.58" y="30.48"/>
-</segment>
-<segment>
+</segment>
+<segment>

Commit message: added a simple pushbutton for increased number of options. I strongly hope that we own smd 2-pin pushbuttons in stock...
Parts:
- added R5: (no value), resistor:R-EU_R0805
- added S1: SWITCH-MOMENTARY-2-SMD-1101NE, SparkFun-Electromechanical:SWITCH-MOMENTARY-2-SMD-1101NE
Connections:
- new net N$8: R5.2, S1.1, U$1.P14_A0_SCK
- net +3V3: now also S1.2
- net GND: now also R5.1
Changed lines of the file:
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@@
 <part name="C4" library="rcl" deviceset="C-EU" device="C0805" value="0.1uF"/>
 <part name="+3V4" library="supply1" deviceset="+3V3" device=""/>
+<part name="S1" library="SparkFun-Electromechanical" deviceset="SWITCH-MOMENTARY-2" device="-SMD-1101NE"/>
+<part name="R5" library="resistor" deviceset="R-EU_" device="R0805"/>
+<part name="GND11" library="supply1" deviceset="GND" device=""/>
+<part name="+3V5" library="supply1" deviceset="+3V3" device=""/>
 </parts>
 <sheets>
@@
 <instance part="C4" gate="G$1" x="-20.32" y="15.24"/>
 <instance part="+3V4" gate="G$1" x="-10.16" y="20.32" rot="R270"/>
+<instance part="S1" gate="G$1" x="114.3" y="73.66" rot="R90"/>
+<instance part="R5" gate="G$1" x="114.3" y="60.96" rot="R90"/>
+<instance part="GND11" gate="1" x="114.3" y="53.34"/>
+<instance part="+3V5" gate="G$1" x="114.3" y="81.28"/>
 </instances>
 <busses>
@@
 <wire x1="-63.5" y1="2.54" x2="-63.5" y2="0" width="0.1524" layer="91"/>
 </segment>
+<segment>
+<pinref part="R5" gate="G$1" pin="1"/>
+<pinref part="GND11" gate="1" pin="GND"/>
+</segment>
 </net>
 <net name="CAP01" class="0">
@@
 <junction x="-20.32" y="20.32"/>
 </segment>
+<segment>
+<pinref part="S1" gate="G$1" pin="2"/>
+<pinref part="+3V5" gate="G$1" pin="+3V3"/>
+</segment>
 </net>
 <net name="SDA" class="0">
@@
 </segment>
 </net>
+<net name="N$8" class="0">
+<segment>
+<pinref part="S1" gate="G$1" pin="1"/>
+<pinref part="R5" gate="G$1" pin="2"/>
+<wire x1="114.3" y1="66.04" x2="114.3" y2="68.58" width="0.1524" layer="91"/>
+<pinref part="U$1" gate="G$1" pin="P14_A0_SCK"/>
+<wire x1="86.36" y1="66.04" x2="114.3" y2="66.04" width="0.1524" layer="91"/>
+</segment>
+</net>

Commit message: new bracelet version! - new teensy only with needed pads - no button - no unnecessary multipliers at the LED - broader circuits - pcb is much smaller
Parts:
- removed R1, R3, R5: (no value), resistor:R-EU_R0805
- removed S1: SWITCH-MOMENTARY-2-SMD-1101NE, SparkFun-Electromechanical:SWITCH-MOMENTARY-2-SMD-1101NE
- removed U$1: TEENSY3, Teensy:TEENSY3
- added U$2: TEENSY3, teensy_minimal:TEENSY3
Connections:
- removed net N$5: LED1.GREEN_A, R2.1
- removed net N$7: R2.2, U$1.P5_TX1
- removed net N$8: R5.2, S1.1, U$1.P14_A0_SCK
- net +3V3: now also U$2.3_3V2; no longer S1.2, U$1.3_3V2
- net BLUETOOTH_TO_TEENSY: now also U$2.P8_DIN_TX3; no longer U$1.P8_DIN_TX3
- net BLUETOOTH_WAKE_HW: now also U$2.P6_CS1; no longer U$1.P6_CS1
- net CAP01: now also U$2.P23_A9_CS2; no longer U$1.P15_A1_CS4
- net CAP02: now also U$2.P0_RX1; no longer U$1.P0_RX1
- net CAP03: now also U$2.P22_A8_CS3; no longer U$1.P16_A2_SCL
- net CAP04: now also U$2.P1_TX1; no longer U$1.P1_TX1
- net CAP05: now also U$2.P15_A1_CS4; no longer U$1.P17_A3_SDA
- net CAP07: now also U$2.P16_A2_SCL; no longer U$1.P23_A9_CS2
- net CAP08: now also U$2.P17_A3_SDA; no longer U$1.P22_A8_CS3
- net GND: now also U$2.GND2; no longer R5.1, U$1.GND2
- net MISO: now also U$2.P12_DIN; no longer U$1.P12_DIN
- net MOSI: now also U$2.P11_DOUT; no longer U$1.P11_DOUT
- net N$2: now also LED1.RED_A, R2.1; no longer R3.2, U$1.P3
- net N$3: now also LED1.BLUE_A, U$2.P5_TX1; no longer R1.2, U$1.P4
- net N$4: now also R2.2, U$2.P4; no longer LED1.RED_A, R1.1
- net N$6: now also LED1.GREEN_A, U$2.P3; no longer LED1.BLUE_A, R3.1
- net SCK: now also U$2.P13_LED_SCK; no longer U$1.P13_LED_SCK
- net SCL: now also U$2.P19_A5_SCL; no longer U$1.P19_A5_SCL
- net SDA: now also U$2.P18_A4_SDA; no longer U$1.P18_A4_SDA
- net SS: now also U$2.P10_CS0_TX2; no longer U$1.P10_CS0_TX2
- net TEENSY_TO_BLUETOOTH: now also U$2.P7_DOUT_RX3; no longer U$1.P7_DOUT_RX3
Other:
- moved on the sheet: R2
